Commit message: updated

File: description/robot_core.xacro (robot description, xacro)
@@ -20,3 +20,10 @@
         <origin xyz="0.1 0 0"/>
     <link name ="chassis">
+        <visual>
+            <origin xyz="0.15 0 0.075"/>
+            <geometry>
+            <box size =" 0.3 0.3 0.15"/>
+            </geometry>
+            <material name="blue"/>
+        </visual>
 </robot>

Commit message: modified:   description/robot_core.xacro 	modified:   package.xml cd '/home/papa-ki-pari/DV/dev_ws/src/minituff'

File: description/robot_core.xacro (robot description, xacro)
@@ -27,3 +27,7 @@
             <material name="blue"/>
         </visual>
+        <collison>
+            <origin xyz="o.15 0 o.075"/>
+            <geometry>
+        </collision>
 </robot>

Commit message: Fix typo in collision element in robot_core.xacro

File: description/robot_core.xacro (robot description, xacro)
@@ -15,19 +15,94 @@
     <link name ="base_link">
     </link>
-    <joint name ="chassis_joint_1"type="fixed">
+    <joint name="chassis_joint" type="fixed">
         <parent link="base_link"/>
-        <child link ="chassis"/>
-        <origin xyz="0.1 0 0"/>
-    <link name ="chassis">
+        <child link="chassis"/>
+        <origin xyz="-0.1 0 0"/>
+    </joint>
+    <link name="chassis">
         <visual>
             <origin xyz="0.15 0 0.075"/>
             <geometry>
-            <box size =" 0.3 0.3 0.15"/>
+                <box size="0.3 0.3 0.15"/>
+            </geometry>
+            <material name="white"/>
+        </visual>
+        <collision>
+            <origin xyz="0.15 0 0.075"/>
+            <geometry>
+                <box size="0.3 0.3 0.15"/>
+            </geometry>
+        </collision>
+        <xacro:inertial_box mass="0.5" x="0.3" y="0.3" z="0.15">
+            <origin xyz="0.15 0 0.075" rpy="0 0 0"/>
+        </xacro:inertial_box>
+    </link>
+//left wheel
+    <joint name="left_wheel_joint" type="continuous">
+        <parent link="base_link"/>
+        <child link="left_wheel"/>
+        <origin xyz="0 0.175 0" rpy="-${pi/2} 0 0" />
+        <axis xyz="0 0 1"/>
+    </joint>
+    <link name="left_wheel">
+        <visual>
+            <geometry>
+                <cylinder radius="0.05" length="0.04"/>
             </geometry>
             <material name="blue"/>
         </visual>
-        <collison>
-            <origin xyz="o.15 0 o.075"/>
+        <collision>
             <geometry>
+                <cylinder radius="0.05" length="0.04"/>
+            </geometry>
         </collision>
+        <xacro:inertial_cylinder mass="0.1" length="0.04" radius="0.05">
+            <origin xyz="0 0 0" rpy="0 0 0"/>
+        </xacro:inertial_cylinder>
+    </link>
+//right wheel
+    <joint name="right_wheel_joint" type="continuous">
+        <parent link="base_link"/>
+        <child link="right_wheel"/>
+        <origin xyz="0 -0.175 0" rpy="${pi/2} 0 0" />
+        <axis xyz="0 0 -1"/>
+    </joint>
+    <link name="right_wheel">
+        <visual>
+            <geometry>
+                <cylinder radius="0.05" length="0.04"/>
+            </geometry>
+            <material name="blue"/>
+        </visual>
+        <collision>
+            <geometry>
+                <cylinder radius="0.05" length="0.04"/>
+            </geometry>
+        </collision>
+        <xacro:inertial_cylinder mass="0.1" length="0.04" radius="0.05">
+            <origin xyz="0 0 0" rpy="0 0 0"/>
+        </xacro:inertial_cylinder>
+    </link>
+    //caster wheel
+    <joint name="caster_wheel_joint" type="fixed">
+        <parent link="chassis"/>
+        <child link="caster_wheel"/>
+        <origin xyz="0.24 0 0"/>
+    </joint>
+    <link name="caster_wheel">
+        <visual>
+            <geometry>
+                <sphere radius="0.05"/>
+            </geometry>
+            <material name="black"/>
+        </visual>
+        <collision>
+            <geometry>
+                <sphere radius="0.05"/>
+            </geometry>
+        </collision>
+        <xacro:inertial_sphere mass="0.1" radius="0.05">
+            <origin xyz="0 0 0" rpy="0 0 0"/>
+        </xacro:inertial_sphere>
+    </link>
 </robot>
